File: CAN_Interjector.kicad_pcb (KiCad board)
At the start: 2 copper layers, 44.4 x 9.5 mm, 5 parts, among them J1 Conn_01x02, J2 Conn_01x02, SW1 SW_DPDT_x2

Commit message: Move the wagos around
Signed-off-by: cfinn <cfinn68916@proton.me>
Parts:
- moved SW1 0.20 mm to (155.0, 102.8)
- moved J2 0.15 mm to (141.1, 104.0)
Changed lines of the file:
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@@
 			(outputformat 1)
 			(mirror no)
-			(drillshape 1)
+			(drillshape 0)
 			(scaleselection 1)
-			(outputdirectory "")
+			(outputdirectory "exports/gbr/")
 		)
 	)
@@
 	(footprint "Library:SW_TL2201EEYA_EWI"
 		(layer "F.Cu")
-		(at 155 103)
+		(at 155 102.8)
 		(tags "TL2201EEYA ")
 		(property "Reference" "SW1"
@@
 	(footprint "TerminalBlock_WAGO:TerminalBlock_WAGO_2601-1102_1x02_P3.50mm_Horizontal"
 		(layer "F.Cu")
-		(at 141.05 103.9 -90)
+		(at 141.05 104.05 -90)
 		(descr "Terminal Block WAGO 2601-1102, 2 pins, pitch 3.5mm, size 8.5x14.5mm, drill diameter 1.2mm, pad diameter 2.3mm, https://www.wago.com/global/pcb-terminal-blocks-and-pluggable-connectors/pcb-terminal-block/p/2601-1102, script-generated using https://gitlab.com/kicad/libraries/kicad-footprint-generator/-/tree/master/scripts/TerminalBlock_WAGO")
 		(tags "THT Terminal Block WAGO 2601-1102 pitch 3.5mm size 8.5x14.5mm drill 1.2mm pad 2.3mm")
@@
 		)
 		(stroke
-			(width 0)
+			(width 0.1)
 			(type solid)
 		)
@@
 		)
 		(stroke
-			(width 0)
+			(width 0.1)
 			(type solid)
 		)
@@
 	)
 	(segment
-		(start 156.25 104.25)
-		(end 169.25 104.25)
+		(start 174.5 104)
+		(end 169.5 104)
 		(width 0.2)
 		(layer "F.Cu")
@@
 	)
 	(segment
-		(start 155 105.5)
-		(end 156.25 104.25)
+		(start 169 104.5)
+		(end 169.5 104)
 		(width 0.2)
 		(layer "F.Cu")
@@
 	)
 	(segment
-		(start 174.5 104)
-		(end 169.5 104)
+		(start 155 105.3)
+		(end 156.05 104.25)
 		(width 0.2)
 		(layer "F.Cu")
@@
 	)
 	(segment
-		(start 169 104.5)
-		(end 169.5 104)
+		(start 156.05 104.25)
+		(end 169.25 104.25)
 		(width 0.2)
 		(layer "F.Cu")
@@
 	)
 	(segment
-		(start 163.149999 105.25)
+		(start 162.949999 105.25)
 		(end 167.25 105.25)
 		(width 0.2)
@@
 	)
 	(segment
-		(start 167.25 105.25)
-		(end 169.5 107.5)
+		(start 152 109.5)
+		(end 158.699999 109.5)
 		(width 0.2)
 		(layer "F.Cu")
@@
 	)
 	(segment
-		(start 160.399999 108)
-		(end 163.149999 105.25)
+		(start 158.699999 109.5)
+		(end 160.399999 107.8)
 		(width 0.2)
 		(layer "F.Cu")
@@
 	)
 	(segment
-		(start 158.899999 109.5)
-		(end 160.399999 108)
+		(start 160.399999 107.8)
+		(end 162.949999 105.25)
 		(width 0.2)
 		(layer "F.Cu")
@@
 	)
 	(segment
-		(start 169 108)
+		(start 167.25 105.25)
 		(end 169.5 107.5)
 		(width 0.2)
@@
 	)
 	(segment
-		(start 174.5 107.5)
+		(start 169 108)
 		(end 169.5 107.5)
 		(width 0.2)
@@
 	)
 	(segment
-		(start 152 109.5)
-		(end 158.899999 109.5)
+		(start 174.5 107.5)
+		(end 169.5 107.5)
 		(width 0.2)
 		(layer "F.Cu")
@@
 	)
 	(segment
-		(start 153.5 105.25)
-		(end 155 103.75)
+		(start 146.05 104.05)
+		(end 141.05 104.05)
 		(width 0.2)
 		(layer "F.Cu")
@@
 	(segment
 		(start 155 103.75)
-		(end 155 103)
+		(end 153.5 105.25)
 		(width 0.2)
 		(layer "F.Cu")
@@
 	)
 	(segment
-		(start 141.05 103.9)
-		(end 146.05 103.9)
+		(start 147.25 105.25)
+		(end 146.05 104.05)
 		(width 0.2)
 		(layer "F.Cu")
@@
 	)
 	(segment
-		(start 155 103)
-		(end 155 102.5)
+		(start 153.5 105.25)
+		(end 147.25 105.25)
 		(width 0.2)
 		(layer "F.Cu")
@@
 	)
 	(segment
-		(start 156.15 101.85)
-		(end 155 103)
+		(start 155 103)
+		(end 155 102.5)
 		(width 0.2)
 		(layer "F.Cu")
@@
 	)
 	(segment
-		(start 147.4 105.25)
-		(end 153.5 105.25)
+		(start 155.95 101.85)
+		(end 155 102.8)
 		(width 0.2)
 		(layer "F.Cu")
@@
 	)
 	(segment
-		(start 146.05 103.9)
-		(end 147.4 105.25)
+		(start 155 102.8)
+		(end 155 103.75)
 		(width 0.2)
 		(layer "F.Cu")
@@
 	(segment
 		(start 163.5 101.85)
-		(end 156.15 101.85)
+		(end 155.95 101.85)
 		(width 0.2)
 		(layer "F.Cu")
@@
 	)
 	(segment
-		(start 146.4 107.4)
-		(end 147.364 106.436)
+		(start 159.263999 106.436)
+		(end 160.399999 105.3)
 		(width 0.2)
 		(layer "F.Cu")
@@
 	)
 	(segment
-		(start 147.364 106.436)
-		(end 159.463999 106.436)
+		(start 159.263999 106.436)
+		(end 152.224936 106.436)
 		(width 0.2)
 		(layer "F.Cu")
@@
 	)
 	(segment
-		(start 141.05 107.4)
-		(end 146.05 107.4)
+		(start 151.110936 107.55)
+		(end 146.05 107.55)
 		(width 0.2)
 		(layer "F.Cu")
@@
 	)
 	(segment
-		(start 159.463999 106.436)
-		(end 160.399999 105.5)
+		(start 146.05 107.4)
+		(end 146.4 107.4)
 		(width 0.2)
 		(layer "F.Cu")
@@
 	)
 	(segment
-		(start 146.05 107.4)
-		(end 146.4 107.4)
+		(start 141.05 107.55)
+		(end 146.05 107.55)
+		(width 0.2)
+		(layer "F.Cu")
+		(net 4)
+	)
+	(segment
+		(start 152.224936 106.436)
+		(end 151.110936 107.55)
 		(width 0.2)
 		(layer "F.Cu")
@@
 	)
 	(segment
-		(start 152 107.85)
+		(start 154.9 107.8)
 		(end 154.85 107.85)
 		(width 0.2)
@@
 	)
 	(segment
-		(start 160.399999 103)
-		(end 163 103)
+		(start 154.85 107.85)
+		(end 152 107.85)
+		(width 0.2)
+		(layer "F.Cu")
+		(net 5)
+	)
+	(segment
+		(start 155 107.8)
+		(end 154.9 107.8)
+		(width 0.2)
+		(layer "F.Cu")
+		(net 5)
+	)
+	(segment
+		(start 161.099999 103.5)
+		(end 160.399999 102.8)
 		(width 0.2)
 		(layer "F.Cu")
@@
 	)
 	(segment
-		(start 163 103)
-		(end 163.5 103.5)
+		(start 163.5 103.5)
+		(end 161.099999 103.5)
 		(width 0.2)
 		(layer "F.Cu")
