File: CAN_Interjector.kicad_pcb (KiCad board)
At the start: 2 copper layers, 44.4 x 9.5 mm, 5 parts, among them J1 Conn_01x02, J2 Conn_01x02, SW1 SW_DPDT_x2

Commit message: Fix stupid encoders
Signed-off-by: cfinn <cfinn68916@proton.me>
Routing:
- net Net-(J1-Pin_1): track 25.9 -> 39.4 mm
- net Net-(SW1B-C): track 3.39 -> 5.58 mm
- net Net-(J1-Pin_2): track 20.4 -> 21.7 mm
Other:
- board text added: "CAN Bus Interjector V0.2"
- board text removed: "CAN Bus Interjector V0.1"
Changed lines of the file:
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@@
 		)
 		(pad "4" thru_hole circle
-			(at 5.399999 5)
+			(at 5.399999 0)
 			(size 1.27 1.27)
 			(drill 0.762)
@@
 		)
 		(pad "6" thru_hole circle
-			(at 5.399999 0)
+			(at 5.399999 5)
 			(size 1.27 1.27)
 			(drill 0.762)
@@
 		)
 	)
-	(gr_text "CAN Bus Interjector V0.1"
-		(at 179.5 110 -0)
+	(gr_text "CAN Bus Interjector V0.2"
+		(at 179.5 110 0)
 		(layer "B.SilkS")
 		(effects
@@
 	)
 	(segment
-		(start 155 105.3)
-		(end 156.05 104.25)
+		(start 156.2 106.5)
+		(end 160.55 106.5)
 		(width 0.2)
-		(layer "F.Cu")
+		(layer "B.Cu")
 		(net 1)
 	)
 	(segment
-		(start 156.05 104.25)
-		(end 169.25 104.25)
+		(start 155 105.3)
+		(end 156.2 106.5)
 		(width 0.2)
-		(layer "F.Cu")
+		(layer "B.Cu")
 		(net 1)
 	)
 	(segment
-		(start 162.949999 105.25)
-		(end 167.25 105.25)
+		(start 163.05 104)
+		(end 169.5 104)
 		(width 0.2)
-		(layer "F.Cu")
-		(net 2)
+		(layer "B.Cu")
+		(net 1)
 	)
 	(segment
-		(start 152 109.5)
-		(end 158.699999 109.5)
+		(start 160.55 106.5)
+		(end 163.05 104)
 		(width 0.2)
-		(layer "F.Cu")
-		(net 2)
+		(layer "B.Cu")
+		(net 1)
 	)
 	(segment
-		(start 158.699999 109.5)
-		(end 160.399999 107.8)
+		(start 164.134867 109.5)
+		(end 166.134867 107.5)
 		(width 0.2)
 		(layer "F.Cu")
@@
 	)
 	(segment
-		(start 160.399999 107.8)
-		(end 162.949999 105.25)
+		(start 152 109.5)
+		(end 164.134867 109.5)
 		(width 0.2)
 		(layer "F.Cu")
@@
 	)
 	(segment
-		(start 167.25 105.25)
+		(start 166.134867 107.5)
 		(end 169.5 107.5)
 		(width 0.2)
@@
 	)
 	(segment
+		(start 170.186338 102.8)
+		(end 160.399999 102.8)
+		(width 0.2)
+		(layer "B.Cu")
+		(net 2)
+	)
+	(segment
+		(start 170.951 106.049)
+		(end 170.951 103.564662)
+		(width 0.2)
+		(layer "B.Cu")
+		(net 2)
+	)
+	(segment
+		(start 169.5 107.5)
+		(end 170.951 106.049)
+		(width 0.2)
+		(layer "B.Cu")
+		(net 2)
+	)
+	(segment
+		(start 170.951 103.564662)
+		(end 170.186338 102.8)
+		(width 0.2)
+		(layer "B.Cu")
+		(net 2)
+	)
+	(segment
 		(start 146.05 104.05)
 		(end 141.05 104.05)
@@
 	)
 	(segment
+		(start 155 102.8)
+		(end 155.95 101.85)
+		(width 0.2)
+		(layer "F.Cu")
+		(net 3)
+	)
+	(segment
 		(start 147.25 105.25)
 		(end 146.05 104.05)
@@
 	)
 	(segment
-		(start 155.95 101.85)
-		(end 155 102.8)
-		(width 0.2)
-		(layer "F.Cu")
-		(net 3)
-	)
-	(segment
 		(start 155 102.8)
 		(end 155 103.75)
@@
 	)
 	(segment
-		(start 163.5 101.85)
-		(end 155.95 101.85)
+		(start 155.95 101.85)
+		(end 163.5 101.85)
 		(width 0.2)
 		(layer "F.Cu")
@@
 	)
 	(segment
-		(start 154.85 107.85)
-		(end 152 107.85)
+		(start 152 107.85)
+		(end 154.95 107.85)
 		(width 0.2)
 		(layer "F.Cu")
@@
 	)
 	(segment
-		(start 161.099999 103.5)
-		(end 160.399999 102.8)
+		(start 154.95 107.85)
+		(end 155 107.8)
 		(width 0.2)
 		(layer "F.Cu")
-		(net 6)
+		(net 5)
 	)
 	(segment
 		(start 163.5 103.5)
-		(end 161.099999 103.5)
+		(end 163.5 104.699999)
+		(width 0.2)
+		(layer "F.Cu")
+		(net 6)
+	)
+	(segment
+		(start 163.5 104.699999)
+		(end 160.399999 107.8)
 		(width 0.2)
 		(layer "F.Cu")
